File: eagle/procesor+pot+display.brd (EAGLE design)
At the start: 52 x 47.9 mm, 26 parts, among them T3 NUD3160, T4 NUD3160

Commit message: modification on Microcontroller PCB
Parts:
- added JP3: (no value), pinhead:1X02/90
- moved JP2 4.02 mm to (16.5, 34.3)
- moved C10 3.81 mm to (47.0, 25.4)
- moved C3 3.81 mm to (47.0, 22.9)
- moved D12 3.81 mm to (41.9, 34.3)
- moved R28 3.81 mm to (19.1, 22.9)
- moved R31 3.81 mm to (16.5, 22.9)
- moved U$2 3.81 mm to (36.8, 36.8)
- moved C1 3.81 mm to (18.7, 6.35)
- moved R25 3.81 mm to (19.1, 10.2)
- moved R26 3.81 mm to (8.89, 10.2)
- moved R29 3.81 mm to (16.5, 10.2)
- moved U$6 3.81 mm to (28.3, 15.2)
- moved C11 3.81 mm to (47.0, 27.9)
- moved J4 3.81 mm to (33.0, 26.7)
- moved JP1 3.81 mm to (41.9, 26.7)
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Connections:
- net 3V3: now also JP2.4
- net GND: now also JP3.2
- net VCC: now also JP3.1; no longer JP2.4
Routing:
- net VCC: track 15.5 -> 35.3 mm
- net 3V3: track 185.7 -> 202.3 mm
- net POTENTIOMETER: track 28.7 -> 31.9 mm
- net TRIAC1: track 21.3 -> 20.0 mm
- net 0V: track 42.9 -> 44.1 mm
- net TRIAC3: track 23.9 -> 22.6 mm
- net GND: track 138.3 -> 137.8 mm, vias 2 -> 4
- net TRIAC2: track 23.0 -> 22.4 mm
Other:
- board size 52 x 47.9 mm -> 52 x 42.9 mm
