File: eagle/procesor+pot+display.sch (EAGLE design)
At the start: 26 parts, among them J4 JP4, T3 NUD3160, T4 NUD3160

Commit message: modification on Microcontroller PCB
Parts:
- added JP3: (no value), pinhead:PINHD-1X2/90
Connections:
- net 3V3: now also JP2.4
- net GND: now also JP3.2
- net VCC: now also JP3.1; no longer JP2.4
Changed lines of the file:
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@@
 <part name="C11" library="adi_v1.6" deviceset="C" device="1206" value="1uF"/>
 <part name="D1" library="adi_v1.6" deviceset="DIODE" device="S1D" value="S1D"/>
+<part name="JP3" library="pinhead" deviceset="PINHD-1X2" device="/90"/>
 </parts>
 <sheets>
@@
 <instance part="C11" gate="C" x="288.544" y="13.462"/>
 <instance part="D1" gate="D$1" x="243.84" y="33.528"/>
+<instance part="JP3" gate="G$1" x="149.86" y="17.78" rot="R180"/>
 </instances>
 <busses>
@@
 <pinref part="C11" gate="C" pin="1"/>
 <wire x1="288.544" y1="16.002" x2="281.432" y2="16.002" width="0.1524" layer="91"/>
+</segment>
+<segment>
+<pinref part="JP2" gate="A" pin="4"/>
+<wire x1="121.92" y1="17.78" x2="127" y2="17.78" width="0.1524" layer="91"/>
+<label x="127" y="17.78" size="1.27" layer="95" xref="yes"/>
 </segment>
 </net>
@@
 <pinref part="C11" gate="C" pin="2"/>
 </segment>
+<segment>
+<pinref part="JP3" gate="G$1" pin="2"/>
+<wire x1="152.4" y1="17.78" x2="160.02" y2="17.78" width="0.1524" layer="91"/>
+<label x="160.02" y="17.78" size="1.27" layer="95" xref="yes"/>
+</segment>
 </net>
 <net name="SEGMENT_A" class="0">
@@
 <net name="VCC" class="0">
 <segment>
-<pinref part="JP2" gate="A" pin="4"/>
-<wire x1="121.92" y1="17.78" x2="127" y2="17.78" width="0.1524" layer="91"/>
-<label x="127" y="17.78" size="1.27" layer="95" xref="yes"/>
-</segment>
-<segment>
 <pinref part="P+8" gate="VCC" pin="VCC"/>
 <wire x1="237.49" y1="15.24" x2="237.49" y2="33.528" width="0.1524" layer="91"/>
@@
 <wire x1="237.49" y1="33.528" x2="241.3" y2="33.528" width="0.1524" layer="91"/>
 </segment>
-</net>
+<segment>
+<pinref part="JP3" gate="G$1" pin="1"/>
+<wire x1="152.4" y1="15.24" x2="160.02" y2="15.24" width="0.1524" layer="91"/>
+<label x="160.02" y="15.24" size="1.27" layer="95" xref="yes"/>
+</segment>
+</net>
